Commit message: Fix robot arm smoothness with S-curve trajectories, kinematics calibration, and gripper orientation

File: src/robot_3dof/urdf/robot_3dof.urdf.xacro (robot description, xacro)
@@ -163,9 +163,9 @@
   <link name="end_effector_link"/>
   <!-- ===================== GRIPPER ===================== -->
-  <!-- Gripper base -->
+  <!-- Gripper base (sits right at the end of link3) -->
   <joint name="gripper_base_joint" type="fixed">
     <parent link="end_effector_link"/>
     <child link="gripper_base_link"/>
-    <origin xyz="0 0 0" rpy="0 0 0"/>
+    <origin xyz="0 0 ${gripper_base_z/2}" rpy="0 0 0"/>
   </joint>
   <link name="gripper_base_link">
@@ -185,9 +185,9 @@
     </collision>
   </link>
-  <!-- Left finger (prismatic along Y, opens outward +Y) -->
+  <!-- Left finger (prismatic along Y, opens outward +Y, extends in +Z) -->
   <joint name="gripper_left_joint" type="prismatic">
     <parent link="gripper_base_link"/>
     <child link="finger_left_link"/>
-    <origin xyz="0 ${finger_y/2} ${-(gripper_base_z/2 + finger_z/2)}" rpy="0 0 0"/>
+    <origin xyz="0 ${finger_y/2} ${gripper_base_z/2 + finger_z/2}" rpy="0 0 0"/>
     <axis xyz="0 1 0"/>
     <limit lower="0.0" upper="0.03" velocity="0.5" effort="20.0"/>
@@ -210,9 +210,9 @@
     </collision>
   </link>
-  <!-- Right finger (mimic of left, moves in -Y) -->
+  <!-- Right finger (mimic of left, moves in -Y, extends in +Z) -->
   <joint name="gripper_right_joint" type="prismatic">
     <parent link="gripper_base_link"/>
     <child link="finger_right_link"/>
-    <origin xyz="0 ${-finger_y/2} ${-(gripper_base_z/2 + finger_z/2)}" rpy="0 0 0"/>
+    <origin xyz="0 ${-finger_y/2} ${gripper_base_z/2 + finger_z/2}" rpy="0 0 0"/>
     <axis xyz="0 1 0"/>
     <limit lower="-0.03" upper="0.0" velocity="0.5" effort="20.0"/>
@@ -236,4 +236,11 @@
     </collision>
   </link>
+  <!-- Grasp Center (virtual reference frame located at the center of the finger pads) -->
+  <joint name="grasp_joint" type="fixed">
+    <parent link="end_effector_link"/>
+    <child link="grasp_link"/>
+    <origin xyz="0 0 ${gripper_base_z + finger_z/2}" rpy="0 0 0"/>
+  </joint>
+  <link name="grasp_link"/>
   <!-- ===================== CAMERA ===================== -->
   <!-- Camera mount (fixed overhead, looking straight down) -->
