Commit message: fix: change joint4 from wrist roll (Z) to wrist pitch (Y) for reliable top-down grasping
ROOT CAUSE: Joint4 rotating around Z (wrist roll) caused the gripper to
tilt sideways when the arm was in a non-vertical pose. One finger would
dip below the table while the other pointed upward, resulting in missed
grasps every time.

FIX:
- URDF: Joint4 axis changed from Z to Y (wrist pitch)
- IK solver: Complete rewrite to Z-Y-Y-Y configuration
  * L1=0.25m (upper arm), L2=0.20m (forearm), L_HAND=0.06m (wrist+gripper)
  * theta4 = pi - (theta2 + theta3) ensures gripper ALWAYS points straight down
  * gripper_pitch is guaranteed 180.0 deg at all reachable positions
- Home position: theta4 now computed as pi-(0.3+0.8)=2.04 rad instead of 0.0
- Place height: lowered from z=0.35 to z=0.30 for better reach

VERIFIED: All 5 test targets reach 0.000mm position error with 180.0 deg pitch

File: src/robot_4dof/urdf/robot_4dof.urdf.xacro (robot description, xacro)
@@ -20,5 +20,5 @@
   <xacro:property name="link3_length" value="0.20"/>
   <xacro:property name="link3_mass" value="0.5"/>
-  <!-- Link4 - Wrist (new 4th DOF: rotation around Z) -->
+  <!-- Link4 - Wrist (new 4th DOF: wrist pitch around Y) -->
   <xacro:property name="link4_radius" value="0.025"/>
   <xacro:property name="link4_height" value="0.03"/>
@@ -159,10 +159,10 @@
     </collision>
   </link>
-  <!-- Link4 - Wrist (4th DOF: rotates around Z for wrist roll) -->
+  <!-- Link4 - Wrist (4th DOF: rotates around Y for wrist pitch) -->
   <joint name="joint4" type="revolute">
     <parent link="link3"/>
     <child link="link4"/>
     <origin xyz="0 0 ${link3_length}" rpy="0 0 0"/>
-    <axis xyz="0 0 1"/>
+    <axis xyz="0 1 0"/>
     <limit lower="${-pi}" upper="${pi}" velocity="3.0" effort="20.0"/>
     <dynamics damping="0.2" friction="0.05"/>
