Commit message: fix(robot_5dof): calibrate table Z to 0.225m, fix wrist roll yaw kinematics, and update README

File: src/robot_5dof/urdf/robot_5dof_gazebo.xacro (robot description, xacro)
@@ -32,9 +32,16 @@
     </material>
   </gazebo>
-  <!-- Link4 - Wrist (NEW: 4th DOF, green) -->
+  <!-- Link4 - Wrist (4th DOF, wrist pitch, green) -->
   <gazebo reference="link4">
     <material>
       <ambient>0.2 0.8 0.3 1</ambient>
       <diffuse>0.2 0.8 0.3 1</diffuse>
+    </material>
+  </gazebo>
+  <!-- Link5 - Wrist Roll (5th DOF, wrist roll, blue) -->
+  <gazebo reference="link5">
+    <material>
+      <ambient>0.2 0.4 0.8 1</ambient>
+      <diffuse>0.2 0.4 0.8 1</diffuse>
     </material>
   </gazebo>
