Commit message: fix(robot_5dof): connect end-effector to link5, enforce wrist pitch limits to prevent folding

File: src/robot_5dof/urdf/robot_5dof.urdf.xacro (robot description, xacro)
@@ -169,5 +169,5 @@
     <origin xyz="0 0 ${link3_length}" rpy="0 0 0"/>
     <axis xyz="0 1 0"/>
-    <limit lower="${-pi}" upper="${pi}" velocity="3.0" effort="20.0"/>
+    <limit lower="${-pi/2}" upper="${pi/2}" velocity="3.0" effort="20.0"/>
     <dynamics damping="0.2" friction="0.05"/>
   </joint>
@@ -195,5 +195,5 @@
     <origin xyz="0 0 ${link4_height}" rpy="0 0 0"/>
     <axis xyz="0 0 1"/>
-    <limit lower="${-pi}" upper="${pi}" velocity="3.0" effort="20.0"/>
+    <limit lower="${-pi/2}" upper="${pi/2}" velocity="3.0" effort="20.0"/>
     <dynamics damping="0.1" friction="0.05"/>
   </joint>
@@ -218,7 +218,7 @@
   <!-- End Effector (reference frame at the tip of wrist link4) -->
   <joint name="end_effector_joint" type="fixed">
-    <parent link="link4"/>
+    <parent link="link5"/>
     <child link="end_effector_link"/>
-    <origin xyz="0 0 ${link4_height}" rpy="0 0 0"/>
+    <origin xyz="0 0 ${link5_height}" rpy="0 0 0"/>
   </joint>
   <link name="end_effector_link"/>

Commit message: fix(grasp): expand joint4 limit to 2.2rad, expand gripper opening to 70mm, increase pre-grasp clearance to 60mm, and clear transit corridor

File: src/robot_5dof/urdf/robot_5dof.urdf.xacro (robot description, xacro)
@@ -169,5 +169,5 @@
     <origin xyz="0 0 ${link3_length}" rpy="0 0 0"/>
     <axis xyz="0 1 0"/>
-    <limit lower="${-pi/2}" upper="${pi/2}" velocity="3.0" effort="20.0"/>
+    <limit lower="-2.2" upper="2.2" velocity="3.0" effort="20.0"/>
     <dynamics damping="0.2" friction="0.05"/>
   </joint>
@@ -252,5 +252,5 @@
     <origin xyz="0 ${finger_y/2} ${gripper_base_z/2 + finger_z/2}" rpy="0 0 0"/>
     <axis xyz="0 1 0"/>
-    <limit lower="0.0" upper="0.03" velocity="0.5" effort="20.0"/>
+    <limit lower="0.0" upper="0.035" velocity="0.5" effort="20.0"/>
     <dynamics damping="0.1"/>
   </joint>
@@ -277,5 +277,5 @@
     <origin xyz="0 ${-finger_y/2} ${gripper_base_z/2 + finger_z/2}" rpy="0 0 0"/>
     <axis xyz="0 1 0"/>
-    <limit lower="-0.03" upper="0.0" velocity="0.5" effort="20.0"/>
+    <limit lower="-0.035" upper="0.0" velocity="0.5" effort="20.0"/>
     <mimic joint="gripper_left_joint" multiplier="-1" offset="0"/>
     <dynamics damping="0.1"/>

File: src/robot_5dof/urdf/robot_5dof_ros2_control.xacro (robot description, xacro)
@@ -55,5 +55,5 @@
       <command_interface name="position">
         <param name="min">0.0</param>
-        <param name="max">0.03</param>
+        <param name="max">0.035</param>
       </command_interface>
       <state_interface name="position"/>
