Commit message: feat: upgrade to 6-DOF robot arm with dual dynamic cameras and evaluate full benchmark matrix

File: src/robot_arm/urdf/robot_arm.urdf.xacro (robot description, xacro)
@@ -1,5 +1,5 @@
 <?xml version="1.0"?>
 <robot xmlns:xacro="http://www.ros.org/wiki/xacro" name="robot_arm">
-  <xacro:arg name="dof" default="5"/>
+  <xacro:arg name="dof" default="6"/>
   <xacro:arg name="use_mesh" default="true"/>
   <!-- ===================== PROPERTIES ===================== -->
@@ -26,8 +26,12 @@
   <xacro:property name="link4_height" value="0.03"/>
   <xacro:property name="link4_mass" value="0.15"/>
-  <!-- Link5 - Wrist Roll (5th DOF: wrist roll around Z) -->
+  <!-- Link5 - Wrist Pitch/Yaw (5th DOF: rotates around X or Z) -->
   <xacro:property name="link5_radius" value="0.025"/>
   <xacro:property name="link5_height" value="0.02"/>
   <xacro:property name="link5_mass" value="0.1"/>
+  <!-- Link6 - Tool Flange / Wrist Roll (6th DOF: tool roll around Z) -->
+  <xacro:property name="link6_radius" value="0.025"/>
+  <xacro:property name="link6_height" value="0.02"/>
+  <xacro:property name="link6_mass" value="0.08"/>
   <!-- Gripper -->
   <xacro:property name="gripper_base_x" value="0.06"/>
@@ -234,5 +238,5 @@
     </link>
   </xacro:if>
-  <xacro:if value="${$(arg dof) >= 5}">
+  <xacro:if value="${$(arg dof) == 5}">
     <joint name="joint5" type="revolute">
       <parent link="link4"/>
@@ -270,4 +274,68 @@
     </link>
   </xacro:if>
+  <xacro:if value="${$(arg dof) >= 6}">
+    <!-- Joint 5 - Wrist Pitch/Yaw (rotates around X) -->
+    <joint name="joint5" type="revolute">
+      <parent link="link4"/>
+      <child link="link5"/>
+      <origin xyz="0 0 ${link4_height}" rpy="0 0 0"/>
+      <axis xyz="1 0 0"/>
+      <limit lower="-2.5" upper="2.5" velocity="3.0" effort="20.0"/>
+      <dynamics damping="0.1" friction="0.05"/>
+    </joint>
+    <link name="link5">
+      <xacro:cylinder_inertia m="${link5_mass}" r="${link5_radius}" h="${link5_height}"/>
+      <visual>
+        <xacro:if value="$(arg use_mesh)">
+          <origin xyz="0 0 0" rpy="0 0 0"/>
+          <geometry>
+            <mesh filename="package://robot_arm/meshes/arm/link5.stl"/>
+          </geometry>
+        </xacro:if>
+        <xacro:unless value="$(arg use_mesh)">
+          <origin xyz="0 0 ${link5_height/2}" rpy="0 0 0"/>
+          <geometry>
+            <cylinder radius="${link5_radius}" length="${link5_height}"/>
+          </geometry>
+        </xacro:unless>
+        <material name="wrist_dark">
+          <color rgba="0.25 0.30 0.35 1.0"/>
+        </material>
+      </visual>
+      <collision>
+        <origin xyz="0 0 ${link5_height/2}" rpy="0 0 0"/>
+        <geometry>
+          <cylinder radius="${link5_radius}" length="${link5_height}"/>
+        </geometry>
+      </collision>
+    </link>
+    <!-- Joint 6 - Tool Flange / Wrist Roll (rotates around Z) -->
+    <joint name="joint6" type="revolute">
+      <parent link="link5"/>
+      <child link="link6"/>
+      <origin xyz="0 0 ${link5_height}" rpy="0 0 0"/>
+      <axis xyz="0 0 1"/>
+      <limit lower="${-pi}" upper="${pi}" velocity="3.0" effort="20.0"/>
+      <dynamics damping="0.1" friction="0.05"/>
+    </joint>
+    <link name="link6">
+      <xacro:cylinder_inertia m="${link6_mass}" r="${link6_radius}" h="${link6_height}"/>
+      <visual>
+        <origin xyz="0 0 ${link6_height/2}" rpy="0 0 0"/>
+        <geometry>
+          <cylinder radius="${link6_radius}" length="${link6_height}"/>
+        </geometry>
+        <material name="flange_dark">
+          <color rgba="0.18 0.22 0.26 1.0"/>
+        </material>
+      </visual>
+      <collision>
+        <origin xyz="0 0 ${link6_height/2}" rpy="0 0 0"/>
+        <geometry>
+          <cylinder radius="${link6_radius}" length="${link6_height}"/>
+        </geometry>
+      </collision>
+    </link>
+  </xacro:if>
   <!-- End Effector (reference frame at the tip of the last link) -->
   <xacro:if value="${$(arg dof) == 3}">
@@ -290,4 +358,11 @@
       <child link="end_effector_link"/>
       <origin xyz="0 0 ${link5_height}" rpy="0 0 0"/>
+    </joint>
+  </xacro:if>
+  <xacro:if value="${$(arg dof) >= 6}">
+    <joint name="end_effector_joint" type="fixed">
+      <parent link="link6"/>
+      <child link="end_effector_link"/>
+      <origin xyz="0 0 ${link6_height}" rpy="0 0 0"/>
     </joint>
   </xacro:if>
@@ -434,4 +509,61 @@
   </joint>
   <link name="camera_optical_link"/>
+  <!-- ===================== DUAL DYNAMIC CAMERAS ===================== -->
+  <!-- Dynamic Camera 1: Wrist Eye-in-Hand Camera (moves with gripper) -->
+  <joint name="camera_wrist_joint" type="fixed">
+    <parent link="gripper_base_link"/>
+    <child link="camera_wrist_link"/>
+    <origin xyz="0.04 0.0 0.02" rpy="0 0.35 0"/>
+  </joint>
+  <link name="camera_wrist_link">
+    <xacro:box_inertia m="${camera_mass}" x="0.025" y="0.05" z="0.02"/>
+    <visual>
+      <geometry>
+        <box size="0.025 0.05 0.02"/>
+      </geometry>
+      <material name="black">
+        <color rgba="0.1 0.1 0.1 1.0"/>
+      </material>
+    </visual>
+    <collision>
+      <geometry>
+        <box size="0.025 0.05 0.02"/>
+      </geometry>
+    </collision>
+  </link>
+  <joint name="camera_wrist_optical_joint" type="fixed">
+    <parent link="camera_wrist_link"/>
+    <child link="camera_wrist_optical_link"/>
+    <origin xyz="0 0 0" rpy="${-pi/2} 0 ${-pi/2}"/>
+  </joint>
+  <link name="camera_wrist_optical_link"/>
+  <!-- Dynamic Camera 2: Arm Turret Tracking Camera (moves with joint1 base yaw) -->
+  <joint name="camera_arm_joint" type="fixed">
+    <parent link="link1"/>
+    <child link="camera_arm_link"/>
+    <origin xyz="0.06 0.0 0.14" rpy="0 0.60 0"/>
+  </joint>
+  <link name="camera_arm_link">
+    <xacro:box_inertia m="${camera_mass}" x="0.03" y="0.05" z="0.025"/>
+    <visual>
+      <geometry>
+        <box size="0.03 0.05 0.025"/>
+      </geometry>
+      <material name="black">
+        <color rgba="0.1 0.1 0.1 1.0"/>
+      </material>
+    </visual>
+    <collision>
+      <geometry>
+        <box size="0.03 0.05 0.025"/>
+      </geometry>
+    </collision>
+  </link>
+  <joint name="camera_arm_optical_joint" type="fixed">
+    <parent link="camera_arm_link"/>
+    <child link="camera_arm_optical_link"/>
+    <origin xyz="0 0 0" rpy="${-pi/2} 0 ${-pi/2}"/>
+  </joint>
+  <link name="camera_arm_optical_link"/>
   <!-- ===================== INCLUDE ros2_control + Gazebo ===================== -->
   <xacro:include filename="$(find robot_arm)/urdf/robot_arm_ros2_control.xacro"/>

File: src/robot_arm/urdf/robot_arm_gazebo.xacro (robot description, xacro)
@@ -47,5 +47,5 @@
   </xacro:if>
   <xacro:if value="${$(arg dof) >= 5}">
-    <!-- Link5 - Wrist Roll -->
+    <!-- Link5 - Wrist Pitch/Roll -->
     <gazebo reference="link5">
       <material>
@@ -56,4 +56,14 @@
     </gazebo>
   </xacro:if>
+  <xacro:if value="${$(arg dof) >= 6}">
+    <!-- Link6 - Flange / Wrist Roll -->
+    <gazebo reference="link6">
+      <material>
+        <ambient>0.25 0.30 0.35 1</ambient>
+        <diffuse>0.25 0.30 0.35 1</diffuse>
+        <specular>0.5 0.5 0.5 1</specular>
+      </material>
+    </gazebo>
+  </xacro:if>
   <!-- Franka Hand (Clean Industrial White) -->
   <gazebo reference="gripper_base_link">
@@ -98,5 +108,5 @@
     </material>
   </gazebo>
-  <!-- ===================== GAZEBO SENSOR: RGBD CAMERA ===================== -->
+  <!-- ===================== SENSOR 1: OVERHEAD SCENE CAMERA ===================== -->
   <gazebo reference="camera_link">
     <sensor name="rgbd_camera" type="rgbd_camera">
@@ -126,3 +136,67 @@
     </sensor>
   </gazebo>
+  <!-- ===================== SENSOR 2: DYNAMIC WRIST EYE-IN-HAND CAMERA ===================== -->
+  <gazebo reference="camera_wrist_link">
+    <material>
+      <ambient>0.1 0.1 0.1 1</ambient>
+      <diffuse>0.1 0.1 0.1 1</diffuse>
+    </material>
+    <sensor name="camera_wrist" type="rgbd_camera">
+      <camera>
+        <horizontal_fov>1.15</horizontal_fov>
+        <image>
+          <width>640</width>
+          <height>480</height>
+          <format>R8G8B8</format>
+        </image>
+        <clip>
+          <near>0.02</near>
+          <far>2.0</far>
+        </clip>
+        <depth_camera>
+          <clip>
+            <near>0.02</near>
+            <far>2.0</far>
+          </clip>
+        </depth_camera>
+      </camera>
+      <always_on>1</always_on>
+      <update_rate>20</update_rate>
+      <visualize>true</visualize>
+      <topic>camera_wrist</topic>
+      <gz_frame_id>camera_wrist_link</gz_frame_id>
+    </sensor>
+  </gazebo>
+  <!-- ===================== SENSOR 3: DYNAMIC ARM TURRET TRACKING CAMERA ===================== -->
+  <gazebo reference="camera_arm_link">
+    <material>
+      <ambient>0.1 0.1 0.1 1</ambient>
+      <diffuse>0.1 0.1 0.1 1</diffuse>
+    </material>
+    <sensor name="camera_arm" type="rgbd_camera">
+      <camera>
+        <horizontal_fov>1.20</horizontal_fov>
+        <image>
+          <width>640</width>
+          <height>480</height>
+          <format>R8G8B8</format>
+        </image>
+        <clip>
+          <near>0.05</near>
+          <far>3.0</far>
+        </clip>
+        <depth_camera>
+          <clip>
+            <near>0.05</near>
+            <far>3.0</far>
+          </clip>
+        </depth_camera>
+      </camera>
+      <always_on>1</always_on>
+      <update_rate>15</update_rate>
+      <visualize>true</visualize>
+      <topic>camera_arm</topic>
+      <gz_frame_id>camera_arm_link</gz_frame_id>
+    </sensor>
+  </gazebo>
 </robot>

File: src/robot_arm/urdf/robot_arm_ros2_control.xacro (robot description, xacro)
@@ -44,5 +44,5 @@
       </joint>
     </xacro:if>
-    <xacro:if value="${$(arg dof) >= 5}">
+    <xacro:if value="${$(arg dof) == 5}">
       <!-- Joint 5 - Wrist Roll (5th DOF) -->
       <joint name="joint5">
@@ -50,4 +50,24 @@
           <param name="min">-1.5708</param>
           <param name="max">1.5708</param>
+        </command_interface>
+        <state_interface name="position"/>
+        <state_interface name="velocity"/>
+      </joint>
+    </xacro:if>
+    <xacro:if value="${$(arg dof) >= 6}">
+      <!-- Joint 5 - Wrist Pitch/Yaw (5th DOF) -->
+      <joint name="joint5">
+        <command_interface name="position">
+          <param name="min">-2.5</param>
+          <param name="max">2.5</param>
+        </command_interface>
+        <state_interface name="position"/>
+        <state_interface name="velocity"/>
+      </joint>
+      <!-- Joint 6 - Tool Flange Roll (6th DOF) -->
+      <joint name="joint6">
+        <command_interface name="position">
+          <param name="min">-3.14159</param>
+          <param name="max">3.14159</param>
         </command_interface>
         <state_interface name="position"/>
